Commit message: Add controller, write README.md

File: urdf/xacro/common/base_link.xacro (robot description, xacro)
@@ -4,4 +4,5 @@
     <xacro:property name="base_high" value="0.2"/>
     <xacro:property name="base_to_ground" value="0.08"/>
+    <xacro:property name="base_m" value="0.5"/>
     <xacro:macro name="base_link">
         <material name="pink">
@@ -9,4 +10,12 @@
         </material>
         <link name="base_link">
+            <inertial>
+                <mass value="${base_m}"/>
+                <inertia ixx="${1/12 * base_m *(base_high * base_high + base_wide * base_wide)}"
+                         ixy="0" ixz="0"
+                         iyy="${1/12 * base_m *(base_length * base_length + base_wide * base_wide)}"
+                         iyz="0" izz="${1/12 * base_m *(base_high * base_high + base_wide * base_wide)}"
+                />
+            </inertial>
             <visual>
                 <origin xyz="0 0 0" rpy="0 0 0" />
@@ -16,4 +25,10 @@
                 <material name="pink"/>
             </visual>
+            <collision>
+                <origin xyz="0 0 0" rpy="0 0 0" />
+                <geometry>
+                    <box size="${base_length} ${base_wide} ${base_high}"/>
+                </geometry>
+            </collision>
         </link>
         <link name="odom">

File: urdf/xacro/common/wheel.xacro (robot description, xacro)
@@ -6,7 +6,17 @@
     <xacro:property name="wheel_radius" value="0.1"/>
     <xacro:property name="wheel_wide" value="0.05"/>
+    <xacro:property name="wheel_m" value="0.2"/>
+    <xacro:property name="mechanical_reduction" value="50"/>
     <xacro:macro name="wheel" params="wheel_name flag_x flag_y">
         <xacro:property name="PI" value="3.14159"/>
         <link name="${wheel_name}_wheel">
+            <inertial>
+                <mass value="${wheel_m}"/>
+                <inertia ixx="${1/12 * wheel_m * (3 * wheel_radius * wheel_radius + wheel_wide * wheel_wide)}"
+                         ixy="0" ixz="0"
+                         iyy="${1/12 * wheel_m * (3 * wheel_radius * wheel_radius + wheel_wide * wheel_wide)}"
+                         iyz="0" izz="${1/2 * wheel_m * wheel_radius * wheel_radius}"
+                />
+            </inertial>
             <visual>
                 <origin xyz="0 0 0" rpy="${PI/2} 0 0"/>
@@ -18,12 +28,36 @@
                 </material>
             </visual>
+            <collision>
+                <origin xyz="0 0 0" rpy="${PI/2} 0 0"/>
+                <geometry>
+                    <cylinder radius="${wheel_radius}" length="${wheel_radius}"/>
+                </geometry>
+            </collision>
         </link>
-        <joint name="base_link2${wheel_name}wheel" type="continuous">
+        <joint name="base_link2${wheel_name}_wheel" type="continuous">
             <parent link="base_link"/>
             <child link="${wheel_name}_wheel"/>
             <origin xyz="${flag_x * base_length / 4} ${flag_y * (wheel_wide + base_wide / 2)}
             ${wheel_radius - base_to_ground - base_high / 2}"/>
-            <anis xyz="0 1 0"/>
+            <axis xyz="0 1 0"/>
         </joint>
     </xacro:macro>
+    <xacro:macro name="wheel_transmission" params="wheel_name">
+        <transmission name="${wheel_name}_wheel_tran">
+            <!--指定传动类型-->
+            <type>transmission_interface/SimpleTransmission</type>
+            <!--传动系统所代表的关节-->
+            <actuator name="${wheel_name}_wheel_motor">
+                <!--可选，指定硬件接口-->
+                <hardwareInterface>hardware_interface/EffortJointInterface</hardwareInterface>
+                <!--可选，指定关节制动器之间机械减速比，并非所有传动系统都需要此标签-->
+                <mechanicalReduction>${mechanical_reduction}</mechanicalReduction>
+            </actuator>
+            <joint name="base_link2${wheel_name}_wheel">
+                <!--指定硬件接口，注意，当在Gazebo中加载此传动系统是，值应为EffortJointInterface-->
+                <!--而在RobotHW中加载此传动系统时，值应为hardware_interface/EffortJointInterface-->
+                <hardwareInterface>hardware_interface/EffortJointInterface</hardwareInterface>
+            </joint>
+        </transmission>
+    </xacro:macro>
 </robot>

File: urdf/xacro/demo01.xacro (robot description, xacro)
@@ -2,8 +2,24 @@
     <xacro:include filename="$(find robot_description)/urdf/xacro/common/base_link.xacro"/>
     <xacro:include filename="$(find robot_description)/urdf/xacro/common/wheel.xacro"/>
-    <xacro:base_link />
-    <xacro:wheel wheel_name="front_left"  flag_x="1" flag_y="1" />
-    <xacro:wheel wheel_name="front_right" flag_x="1" flag_y="-1" />
+    <xacro:base_link/>
+    <xacro:wheel wheel_name="front_left"  flag_x="1"  flag_y="1" />
+    <xacro:wheel wheel_name="front_right" flag_x="1"  flag_y="-1" />
     <xacro:wheel wheel_name="back_left"   flag_x="-1" flag_y="1" />
     <xacro:wheel wheel_name="back_right"  flag_x="-1" flag_y="-1" />
+    <xacro:wheel_transmission wheel_name="front_left" />
+    <xacro:wheel_transmission wheel_name="front_right"/>
+    <xacro:wheel_transmission wheel_name="back_left"  />
+    <xacro:wheel_transmission wheel_name="back_right" />
+<!--    添加gazebo_ros_control插件-->
+    <gazebo>
+<!--        <plugin name="ros_control" filename="libgazebo_ros_control.so">-->
+<!--        <plugin name="gazebo_ros_control" filename="libgazebo_ros_control.so">-->
+<!--            <robotNamespace>/robot_description</robotNamespace>-->
+<!--            <robotSimType>gazebo_ros_control/DefaultRobotHWSim</robotSimType>-->
+<!--        </plugin>-->
+        <plugin name="rm_ros_control" filename="librm_robot_hw_sim.so">
+            <robotNamespace>/</robotNamespace>
+            <robotSimType>rm_gazebo/RmRobotHWSim</robotSimType>
+        </plugin>
+    </gazebo>
 </robot>
